File: hardware/Motor/Motors.brd (EAGLE design)
At the start: 59 x 48 mm, 34 parts, among them IC1 MC33269ST, Q1 BSS138, Q2 BSS138, U1 DRV8884PWPR, U2 PHOTON_WITH_HEADERS, U3 LS7083N-S

Commit message: Cumulative changes: adding light sources, boards, firmwares, construction details
Parts:
- removed DC1: Power Connector, Spectron2:POWERSUPPLY_DC-21MM
- added J1: +12V, WEIDMULLER-PM5.08_2_90BLK:WEIDMULLER_PM5.08_2
Connections:
- net GND: now also J1.1; no longer DC1.1, DC1.3
- net VIN: now also J1.2; no longer DC1.2
Changed lines of the file:
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@@
 <?xml version="1.0" encoding="utf-8"?>
 <!DOCTYPE eagle SYSTEM "eagle.dtd">
-<eagle version="7.7.0">
+<eagle version="8.0.1">
 <drawing>
 <settings>
@@
 <layers>
 <layer number="1" name="Top" color="4" fill="1" visible="yes" active="yes"/>
+<layer number="2" name="Route2" color="1" fill="3" visible="no" active="no"/>
+<layer number="3" name="Route3" color="4" fill="3" visible="no" active="no"/>
+<layer number="4" name="Route4" color="1" fill="4" visible="no" active="no"/>
+<layer number="5" name="Route5" color="4" fill="4" visible="no" active="no"/>
+<layer number="6" name="Route6" color="1" fill="8" visible="no" active="no"/>
+<layer number="7" name="Route7" color="4" fill="8" visible="no" active="no"/>
+<layer number="8" name="Route8" color="1" fill="2" visible="no" active="no"/>
+<layer number="9" name="Route9" color="4" fill="2" visible="no" active="no"/>
+<layer number="10" name="Route10" color="1" fill="7" visible="no" active="no"/>
+<layer number="11" name="Route11" color="4" fill="7" visible="no" active="no"/>
+<layer number="12" name="Route12" color="1" fill="5" visible="no" active="no"/>
+<layer number="13" name="Route13" color="4" fill="5" visible="no" active="no"/>
+<layer number="14" name="Route14" color="1" fill="6" visible="no" active="no"/>
+<layer number="15" name="Route15" color="4" fill="6" visible="no" active="no"/>
 <layer number="16" name="Bottom" color="1" fill="1" visible="yes" active="yes"/>
 <layer number="17" name="Pads" color="2" fill="1" visible="yes" active="yes"/>
@@
 <attribute name="VALUE" x="6.66" y="20.52" size="0.8128" layer="28" rot="MR270"/>
 </element>
-<element name="DC1" library="Spectron2" package="POWERSUPPLY_DC-21MM" value="Power Connector" x="5.11" y="11.28" smashed="yes" rot="R90">
-<attribute name="NAME" x="9.46" y="3.63" size="0.8128" layer="25" ratio="5" rot="R180"/>
-<attribute name="VALUE" x="1.54" y="15.83" size="0.8128" layer="27" ratio="5"/>
-</element>
 <element name="FRAME1" library="SparkFun-Aesthetics" package="CREATIVE_COMMONS" value="FRAME-LETTER" x="3.96" y="40.12"/>
 <element name="IC1" library="Spectron" package="SOT223" value="MC33269ST" x="45.74" y="10.09" rot="R270"/>
@@
 <attribute name="VALUE" x="31.135" y="17.46" size="0.8128" layer="28" rot="MR0"/>
 </element>
+<element name="J1" library="WEIDMULLER-PM5.08_2_90BLK" package="WEIDMULLER_PM5.08_2" value="+12V" x="6" y="10.7">
+<attribute name="SUPPLIER" value="WEIDMULLER " x="6" y="10.7" size="1.778" layer="27" display="off"/>
+<attribute name="OC_FARNELL" value="1131855 " x="6" y="10.7" size="1.778" layer="27" display="off"/>
+<attribute name="PACKAGE" value="TH-R/A" x="6" y="10.7" size="1.778" layer="27" display="off"/>
+<attribute name="MPN" value="PM5.08/2/90 BLK" x="6" y="10.7" size="1.778" layer="27" display="off"/>
+<attribute name="OC_NEWARK" value="26M1980 " x="6" y="10.7" size="1.778" layer="27" display="off"/>
+</element>
 </elements>
 <signals>
@@
 </signal>
 <signal name="VIN">
-<contactref element="DC1" pad="2"/>
 <contactref element="IC1" pad="3"/>
 <contactref element="C8" pad="+"/>
@@
 <vertex x="14.1732" y="12.192"/>
 <vertex x="13.2588" y="13.1064"/>
-<vertex x="10.668" y="13.1064"/>
-<vertex x="9.4488" y="11.8872"/>
-<vertex x="9.4488" y="10.5156"/>
-<vertex x="11.43" y="8.5344"/>
-<vertex x="11.43" y="4.2672"/>
+<vertex x="7.668" y="13.1064"/>
+<vertex x="6.4488" y="11.8872"/>
+<vertex x="6.4488" y="9.5156"/>
+<vertex x="9.43" y="7.5344"/>
+<vertex x="9.43" y="5.2672"/>
 <vertex x="14.0208" y="1.6764"/>
 <vertex x="26.1056" y="1.6764"/>
@@
 <vertex x="39.8" y="9"/>
 </polygon>
+<contactref element="J1" pad="2"/>
 </signal>
 <signal name="GND">
@@
 <contactref element="U1" pad="6"/>
 <contactref element="U1" pad="9"/>
-<contactref element="DC1" pad="3"/>
-<contactref element="DC1" pad="1"/>
 <contactref element="IC1" pad="1"/>
 <contactref element="C8" pad="-"/>
@@
 <via x="11" y="28" extent="1-16" drill="0.3302" diameter="0.1778"/>
 <via x="13" y="26" extent="1-16" drill="0.3302" diameter="0.1778"/>
+<contactref element="J1" pad="1"/>
 </signal>
 <signal name="+5V">
