File: hardware/Spectrometer/Spectron2.brd (EAGLE design)
At the start: 70 x 54 mm, 69 parts, among them U1 REF192, U10 ADP7142-2.5, U11 REF195, U12 TLV809, U13 ADG821, U14 ADG3304, U15 LM2662, U16 PHOTON_WITH_HEADERS, U2 ADG1604, U3 ADP7142-5, U4 AD8031, U5 REF193, U6 ADA4841, U7 ADP7142-5, U8 AD7980, U9 REF198

Commit message: Cumulative changes: adding light sources, boards, firmwares, construction details
Parts:
- removed DC1: POWERSUPPLY_DC21MMX, Spectron:POWERSUPPLY_DC-21MM
- added J1: +5V, WEIDMULLER-PM5.08_2_90BLK:WEIDMULLER_PM5.08_2
- moved FRAME1 2.92 mm to (-0.04, 0.23)
Connections:
- net GND: now also J1.1; no longer DC1.1, DC1.3
- net N$11: now also J1.2; no longer DC1.2
Routing:
- net VIN: track 39.2 -> 37.7 mm
Changed lines of the file:
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@@
 <?xml version="1.0" encoding="utf-8"?>
 <!DOCTYPE eagle SYSTEM "eagle.dtd">
-<eagle version="7.7.0">
+<eagle version="8.0.1">
 <drawing>
 <settings>
@@
 <layers>
 <layer number="1" name="Top" color="4" fill="1" visible="yes" active="yes"/>
+<layer number="2" name="Route2" color="1" fill="3" visible="no" active="no"/>
+<layer number="3" name="Route3" color="4" fill="3" visible="no" active="no"/>
+<layer number="4" name="Route4" color="1" fill="4" visible="no" active="no"/>
+<layer number="5" name="Route5" color="4" fill="4" visible="no" active="no"/>
+<layer number="6" name="Route6" color="1" fill="8" visible="no" active="no"/>
+<layer number="7" name="Route7" color="4" fill="8" visible="no" active="no"/>
+<layer number="8" name="Route8" color="1" fill="2" visible="no" active="no"/>
+<layer number="9" name="Route9" color="4" fill="2" visible="no" active="no"/>
+<layer number="10" name="Route10" color="1" fill="7" visible="no" active="no"/>
+<layer number="11" name="Route11" color="4" fill="7" visible="no" active="no"/>
+<layer number="12" name="Route12" color="1" fill="5" visible="no" active="no"/>
+<layer number="13" name="Route13" color="4" fill="5" visible="no" active="no"/>
+<layer number="14" name="Route14" color="1" fill="6" visible="no" active="no"/>
+<layer number="15" name="Route15" color="4" fill="6" visible="no" active="no"/>
 <layer number="16" name="Bottom" color="1" fill="1" visible="yes" active="yes"/>
 <layer number="17" name="Pads" color="2" fill="1" visible="yes" active="yes"/>
@@
 <attribute name="NAME" x="16.299" y="13.446" size="0.8128" layer="25"/>
 </element>
-<element name="DC1" library="Spectron" package="POWERSUPPLY_DC-21MM" value="POWERSUPPLY_DC21MMX" x="5.08" y="11.23" smashed="yes" rot="R90">
-<attribute name="NAME" x="10.16" y="13.77" size="1.016" layer="25" ratio="5" rot="R180"/>
-</element>
-<element name="FRAME1" library="SparkFun-Aesthetics" package="CREATIVE_COMMONS" value="FRAME-LEDGER" x="-2.54" y="-1.27"/>
+<element name="FRAME1" library="SparkFun-Aesthetics" package="CREATIVE_COMMONS" value="FRAME-LEDGER" x="-0.04" y="0.23"/>
 <element name="JP1" library="SparkFun-Connectors" package="1X08" value="C12666/C12880" x="38.1" y="19.685" smashed="yes" rot="MR90">
 <attribute name="PROD_ID" value="CONN-08438" x="38.1" y="19.685" size="1.778" layer="28" rot="MR90" display="off"/>
@@
 <attribute name="VALUE" x="45.74" y="19.235" size="1.27" layer="28" rot="MR270"/>
 </element>
+<element name="J1" library="WEIDMULLER-PM5.08_2_90BLK" package="WEIDMULLER_PM5.08_2" value="+5V" x="9" y="8.6" rot="R90">
+<attribute name="SUPPLIER" value="WEIDMULLER " x="9" y="8.6" size="1.778" layer="27" rot="R90" display="off"/>
+<attribute name="OC_FARNELL" value="1131855 " x="9" y="8.6" size="1.778" layer="27" rot="R90" display="off"/>
+<attribute name="PACKAGE" value="TH-R/A" x="9" y="8.6" size="1.778" layer="27" rot="R90" display="off"/>
+<attribute name="MPN" value="PM5.08/2/90 BLK" x="9" y="8.6" size="1.778" layer="27" rot="R90" display="off"/>
+<attribute name="OC_NEWARK" value="26M1980 " x="9" y="8.6" size="1.778" layer="27" rot="R90" display="off"/>
+</element>
 </elements>
 <signals>
@@
 </signal>
 <signal name="GND">
-<contactref element="DC1" pad="1"/>
-<contactref element="DC1" pad="3"/>
 <contactref element="U8" pad="5"/>
 <contactref element="U8" pad="4"/>
@@
 <via x="19.035" y="35.055" extent="1-16" drill="0.3302" diameter="0.1778"/>
 <via x="21.035" y="35.055" extent="1-16" drill="0.3302" diameter="0.1778"/>
+<contactref element="J1" pad="1"/>
 </signal>
 <signal name="3.3V">
@@
 <contactref element="C29" pad="2"/>
 <contactref element="U16" pad="1"/>
-<contactref element="D2" pad="C"/>
-<contactref element="U15" pad="3"/>
-<contactref element="D1" pad="A"/>
-<wire x1="18.918" y1="12.192" x2="18.918" y2="13.721" width="1.27" layer="1"/>
 <wire x1="18.918" y1="13.721" x2="17.78" y2="15.24" width="1.27" layer="1"/>
 <wire x1="17.78" y1="15.24" x2="7.62" y2="15.24" width="1.27" layer="1"/>
@@
 </polygon>
 <via x="6.223" y="23.495" extent="1-16" drill="0.3302" diameter="0.1778"/>
+<contactref element="D2" pad="C"/>
+<contactref element="U15" pad="3"/>
+<contactref element="D1" pad="A"/>
 </signal>
 <signal name="N$2">
@@
 </signal>
 <signal name="N$11">
-<contactref element="DC1" pad="2"/>
 <contactref element="D2" pad="A"/>
 <polygon width="0.1524" layer="1" thermals="no">
 <vertex x="15.875" y="13.081"/>
-<vertex x="10.668" y="13.081"/>
-<vertex x="9.525" y="11.938"/>
-<vertex x="9.525" y="10.414"/>
-<vertex x="10.668" y="9.271"/>
+<vertex x="7.668" y="13.081"/>
+<vertex x="6.525" y="11.938"/>
+<vertex x="6.525" y="10.414"/>
+<vertex x="7.668" y="9.271"/>
 <vertex x="12.319" y="9.271"/>
 <vertex x="13.335" y="10.287"/>
@@
 <vertex x="15.875" y="11.557"/>
 </polygon>
+<contactref element="J1" pad="2"/>
 </signal>
 <signal name="N$8">
